File: HARDWARE/KiCad/PCBTrack/PCBTrack.kicad_pcb (KiCad board)
At the start: 2 copper layers, 45 x 56 mm, 9 parts

Commit message: add PDF
Parts:
- added REF**: PinHeader_1x03_P2.00mm_Horizontal, Connector_PinHeader_2.00mm:PinHeader_1x03_P2.00mm_Horizontal, F.Cu at (106.0, 158.5)
- added REF**: PinHeader_1x03_P2.00mm_Horizontal, Connector_PinHeader_2.00mm:PinHeader_1x03_P2.00mm_Horizontal, F.Cu at (28.0, 158.5)
- added REF**: PinHeader_1x03_P1.27mm_Horizontal, Connector_PinHeader_1.27mm:PinHeader_1x03_P1.27mm_Horizontal, F.Cu at (28.0, 166.0)
- added REF**: PinHeader_1x03_P1.00mm_Horizontal, Connector_PinHeader_1.00mm:PinHeader_1x03_P1.00mm_Horizontal, F.Cu at (28.0, 172.8)
- added REF**: DIP-4_W10.16mm_LongPads, Package_DIP:DIP-4_W10.16mm_LongPads, F.Cu at (67.0, 191.0)
- added REF**: DIP-4_W10.16mm, Package_DIP:DIP-4_W10.16mm, F.Cu at (58.0, 191.0)
- added REF**: DIP-4_W7.62mm_Socket, Package_DIP:DIP-4_W7.62mm_Socket, F.Cu at (40.0, 190.0)
- added REF**: DIP-4_W7.62mm_LongPads, Package_DIP:DIP-4_W7.62mm_LongPads, F.Cu at (31.0, 190.0)
- added REF**: DIP-4_W7.62mm_Socket_LongPads, Package_DIP:DIP-4_W7.62mm_Socket_LongPads, F.Cu at (49.0, 190.0)
- added REF**: DIP-4_W7.62mm, Package_DIP:DIP-4_W7.62mm, F.Cu at (22.0, 190.0)
- added REF**: PinHeader_1x03_P2.00mm_Horizontal, Connector_PinHeader_2.00mm:PinHeader_1x03_P2.00mm_Horizontal, F.Cu at (268.5, 95.0)
- added REF**: PinHeader_1x03_P1.27mm_Horizontal, Connector_PinHeader_1.27mm:PinHeader_1x03_P1.27mm_Horizontal, F.Cu at (106.0, 166.0)
- added REF**: PinHeader_1x03_P1.27mm_Horizontal, Connector_PinHeader_1.27mm:PinHeader_1x03_P1.27mm_Horizontal, F.Cu at (261.0, 95.0)
- added REF**: PinHeader_1x03_P1.00mm_Horizontal, Connector_PinHeader_1.00mm:PinHeader_1x03_P1.00mm_Horizontal, F.Cu at (254.2, 95.0)
- added REF**: DIP-4_W10.16mm_LongPads, Package_DIP:DIP-4_W10.16mm_LongPads, F.Cu at (236.0, 134.0)
- added REF**: DIP-4_W10.16mm, Package_DIP:DIP-4_W10.16mm, F.Cu at (236.0, 125.0)
- added REF**: DIP-4_W7.62mm_Socket, Package_DIP:DIP-4_W7.62mm_Socket, F.Cu at (237.0, 107.0)
- added REF**: DIP-4_W7.62mm_LongPads, Package_DIP:DIP-4_W7.62mm_LongPads, F.Cu at (237.0, 98.0)
- added REF**: DIP-4_W7.62mm_Socket_LongPads, Package_DIP:DIP-4_W7.62mm_Socket_LongPads, F.Cu at (237.0, 116.0)
- added REF**: DIP-4_W7.62mm, Package_DIP:DIP-4_W7.62mm, F.Cu at (237.0, 89.0)
- added REF**: PinHeader_1x03_P2.00mm_Horizontal, Connector_PinHeader_2.00mm:PinHeader_1x03_P2.00mm_Horizontal, F.Cu at (268.5, 28.0)
- added REF**: PinHeader_1x03_P1.27mm_Horizontal, Connector_PinHeader_1.27mm:PinHeader_1x03_P1.27mm_Horizontal, F.Cu at (261.0, 28.0)
- added REF**: PinHeader_1x03_P1.00mm_Horizontal, Connector_PinHeader_1.00mm:PinHeader_1x03_P1.00mm_Horizontal, F.Cu at (106.0, 172.8)
- added REF**: PinHeader_1x03_P1.00mm_Horizontal, Connector_PinHeader_1.00mm:PinHeader_1x03_P1.00mm_Horizontal, F.Cu at (254.2, 28.0)
- added REF**: DIP-4_W10.16mm_LongPads, Package_DIP:DIP-4_W10.16mm_LongPads, F.Cu at (236.0, 67.0)
- added REF**: DIP-4_W10.16mm, Package_DIP:DIP-4_W10.16mm, F.Cu at (236.0, 58.0)
- added REF**: DIP-4_W7.62mm_Socket, Package_DIP:DIP-4_W7.62mm_Socket, F.Cu at (237.0, 40.0)
- added REF**: DIP-4_W7.62mm_LongPads, Package_DIP:DIP-4_W7.62mm_LongPads, F.Cu at (237.0, 31.0)
- added REF**: DIP-4_W7.62mm_Socket_LongPads, Package_DIP:DIP-4_W7.62mm_Socket_LongPads, F.Cu at (237.0, 49.0)
- added REF**: DIP-4_W7.62mm, Package_DIP:DIP-4_W7.62mm, F.Cu at (237.0, 22.0)
- added REF**: PinHeader_1x03_P2.00mm_Horizontal, Connector_PinHeader_2.00mm:PinHeader_1x03_P2.00mm_Horizontal, F.Cu at (215.5, 95.0)
- added REF**: PinHeader_1x03_P1.27mm_Horizontal, Connector_PinHeader_1.27mm:PinHeader_1x03_P1.27mm_Horizontal, F.Cu at (208.0, 95.0)
- added REF**: PinHeader_1x03_P1.00mm_Horizontal, Connector_PinHeader_1.00mm:PinHeader_1x03_P1.00mm_Horizontal, F.Cu at (201.2, 95.0)
- added REF**: DIP-4_W10.16mm_LongPads, Package_DIP:DIP-4_W10.16mm_LongPads, F.Cu at (145.0, 191.0)
- added REF**: DIP-4_W10.16mm_LongPads, Package_DIP:DIP-4_W10.16mm_LongPads, F.Cu at (183.0, 134.0)
- added REF**: DIP-4_W10.16mm, Package_DIP:DIP-4_W10.16mm, F.Cu at (183.0, 125.0)
- added REF**: DIP-4_W7.62mm_Socket, Package_DIP:DIP-4_W7.62mm_Socket, F.Cu at (184.0, 107.0)
- added REF**: DIP-4_W7.62mm_LongPads, Package_DIP:DIP-4_W7.62mm_LongPads, F.Cu at (184.0, 98.0)
- added REF**: DIP-4_W7.62mm_Socket_LongPads, Package_DIP:DIP-4_W7.62mm_Socket_LongPads, F.Cu at (184.0, 116.0)
- added REF**: DIP-4_W7.62mm, Package_DIP:DIP-4_W7.62mm, F.Cu at (184.0, 89.0)
- added REF**: PinHeader_1x03_P2.00mm_Horizontal, Connector_PinHeader_2.00mm:PinHeader_1x03_P2.00mm_Horizontal, F.Cu at (215.5, 28.0)
- added REF**: PinHeader_1x03_P1.27mm_Horizontal, Connector_PinHeader_1.27mm:PinHeader_1x03_P1.27mm_Horizontal, F.Cu at (208.0, 28.0)
- added REF**: PinHeader_1x03_P1.00mm_Horizontal, Connector_PinHeader_1.00mm:PinHeader_1x03_P1.00mm_Horizontal, F.Cu at (201.2, 28.0)
- added REF**: DIP-4_W10.16mm_LongPads, Package_DIP:DIP-4_W10.16mm_LongPads, F.Cu at (183.0, 67.0)
- added REF**: DIP-4_W10.16mm, Package_DIP:DIP-4_W10.16mm, F.Cu at (136.0, 191.0)
- added REF**: DIP-4_W10.16mm, Package_DIP:DIP-4_W10.16mm, F.Cu at (183.0, 58.0)
- added REF**: DIP-4_W7.62mm_Socket, Package_DIP:DIP-4_W7.62mm_Socket, F.Cu at (184.0, 40.0)
- added REF**: DIP-4_W7.62mm_LongPads, Package_DIP:DIP-4_W7.62mm_LongPads, F.Cu at (184.0, 31.0)
- added REF**: DIP-4_W7.62mm_Socket_LongPads, Package_DIP:DIP-4_W7.62mm_Socket_LongPads, F.Cu at (184.0, 49.0)
- added REF**: DIP-4_W7.62mm, Package_DIP:DIP-4_W7.62mm, F.Cu at (184.0, 22.0)
- added REF**: PinHeader_1x03_P2.00mm_Horizontal, Connector_PinHeader_2.00mm:PinHeader_1x03_P2.00mm_Horizontal, F.Cu at (162.5, 95.0)
- added REF**: PinHeader_1x03_P1.27mm_Horizontal, Connector_PinHeader_1.27mm:PinHeader_1x03_P1.27mm_Horizontal, F.Cu at (155.0, 95.0)
- added REF**: PinHeader_1x03_P1.00mm_Horizontal, Connector_PinHeader_1.00mm:PinHeader_1x03_P1.00mm_Horizontal, F.Cu at (148.2, 95.0)
- added REF**: DIP-4_W10.16mm_LongPads, Package_DIP:DIP-4_W10.16mm_LongPads, F.Cu at (130.0, 134.0)
- added REF**: DIP-4_W10.16mm, Package_DIP:DIP-4_W10.16mm, F.Cu at (130.0, 125.0)
- added REF**: DIP-4_W7.62mm_Socket, Package_DIP:DIP-4_W7.62mm_Socket, F.Cu at (118.0, 190.0)
- added REF**: DIP-4_W7.62mm_Socket, Package_DIP:DIP-4_W7.62mm_Socket, F.Cu at (131.0, 107.0)
- added REF**: DIP-4_W7.62mm_LongPads, Package_DIP:DIP-4_W7.62mm_LongPads, F.Cu at (131.0, 98.0)
- added REF**: DIP-4_W7.62mm_Socket_LongPads, Package_DIP:DIP-4_W7.62mm_Socket_LongPads, F.Cu at (131.0, 116.0)
- added REF**: DIP-4_W7.62mm, Package_DIP:DIP-4_W7.62mm, F.Cu at (131.0, 89.0)
- added REF**: PinHeader_1x03_P2.00mm_Horizontal, Connector_PinHeader_2.00mm:PinHeader_1x03_P2.00mm_Horizontal, F.Cu at (162.5, 28.0)
- added REF**: PinHeader_1x03_P1.27mm_Horizontal, Connector_PinHeader_1.27mm:PinHeader_1x03_P1.27mm_Horizontal, F.Cu at (155.0, 28.0)
- added REF**: PinHeader_1x03_P1.00mm_Horizontal, Connector_PinHeader_1.00mm:PinHeader_1x03_P1.00mm_Horizontal, F.Cu at (148.2, 28.0)
- added REF**: DIP-4_W10.16mm_LongPads, Package_DIP:DIP-4_W10.16mm_LongPads, F.Cu at (130.0, 67.0)
- added REF**: DIP-4_W10.16mm, Package_DIP:DIP-4_W10.16mm, F.Cu at (130.0, 58.0)
- added REF**: DIP-4_W7.62mm_Socket, Package_DIP:DIP-4_W7.62mm_Socket, F.Cu at (131.0, 40.0)
- added REF**: DIP-4_W7.62mm_LongPads, Package_DIP:DIP-4_W7.62mm_LongPads, F.Cu at (109.0, 190.0)
- added REF**: DIP-4_W7.62mm_LongPads, Package_DIP:DIP-4_W7.62mm_LongPads, F.Cu at (131.0, 31.0)
- added REF**: DIP-4_W7.62mm_Socket_LongPads, Package_DIP:DIP-4_W7.62mm_Socket_LongPads, F.Cu at (131.0, 49.0)
- added REF**: DIP-4_W7.62mm, Package_DIP:DIP-4_W7.62mm, F.Cu at (131.0, 22.0)
- added REF**: PinHeader_1x03_P2.00mm_Horizontal, Connector_PinHeader_2.00mm:PinHeader_1x03_P2.00mm_Horizontal, F.Cu at (108.5, 95.0)
- added REF**: PinHeader_1x03_P1.27mm_Horizontal, Connector_PinHeader_1.27mm:PinHeader_1x03_P1.27mm_Horizontal, F.Cu at (101.0, 95.0)
- added REF**: PinHeader_1x03_P1.00mm_Horizontal, Connector_PinHeader_1.00mm:PinHeader_1x03_P1.00mm_Horizontal, F.Cu at (94.2, 95.0)
- added REF**: DIP-4_W10.16mm_LongPads, Package_DIP:DIP-4_W10.16mm_LongPads, F.Cu at (76.0, 134.0)
- added REF**: DIP-4_W10.16mm, Package_DIP:DIP-4_W10.16mm, F.Cu at (76.0, 125.0)
- added REF**: DIP-4_W7.62mm_Socket, Package_DIP:DIP-4_W7.62mm_Socket, F.Cu at (77.0, 107.0)
- added REF**: DIP-4_W7.62mm_LongPads, Package_DIP:DIP-4_W7.62mm_LongPads, F.Cu at (77.0, 98.0)
- added REF**: DIP-4_W7.62mm_Socket_LongPads, Package_DIP:DIP-4_W7.62mm_Socket_LongPads, F.Cu at (127.0, 190.0)
- added REF**: DIP-4_W7.62mm_Socket_LongPads, Package_DIP:DIP-4_W7.62mm_Socket_LongPads, F.Cu at (77.0, 116.0)
- added REF**: DIP-4_W7.62mm, Package_DIP:DIP-4_W7.62mm, F.Cu at (77.0, 89.0)
- added REF**: PinHeader_1x03_P2.00mm_Horizontal, Connector_PinHeader_2.00mm:PinHeader_1x03_P2.00mm_Horizontal, F.Cu at (109.5, 28.0)
- added REF**: PinHeader_1x03_P1.27mm_Horizontal, Connector_PinHeader_1.27mm:PinHeader_1x03_P1.27mm_Horizontal, F.Cu at (102.0, 28.0)
- added REF**: PinHeader_1x03_P1.00mm_Horizontal, Connector_PinHeader_1.00mm:PinHeader_1x03_P1.00mm_Horizontal, F.Cu at (95.2, 28.0)
- added REF**: DIP-4_W10.16mm_LongPads, Package_DIP:DIP-4_W10.16mm_LongPads, F.Cu at (77.0, 67.0)
- added REF**: DIP-4_W10.16mm, Package_DIP:DIP-4_W10.16mm, F.Cu at (77.0, 58.0)
- added REF**: DIP-4_W7.62mm_Socket, Package_DIP:DIP-4_W7.62mm_Socket, F.Cu at (78.0, 40.0)
- added REF**: DIP-4_W7.62mm_LongPads, Package_DIP:DIP-4_W7.62mm_LongPads, F.Cu at (78.0, 31.0)
- added REF**: DIP-4_W7.62mm_Socket_LongPads, Package_DIP:DIP-4_W7.62mm_Socket_LongPads, F.Cu at (78.0, 49.0)
- added REF**: DIP-4_W7.62mm, Package_DIP:DIP-4_W7.62mm, F.Cu at (100.0, 190.0)
- added REF**: DIP-4_W7.62mm, Package_DIP:DIP-4_W7.62mm, F.Cu at (78.0, 22.0)
- added REF**: PinHeader_1x03_P2.00mm_Horizontal, Connector_PinHeader_2.00mm:PinHeader_1x03_P2.00mm_Horizontal, F.Cu at (55.5, 95.0)
- added REF**: PinHeader_1x03_P1.27mm_Horizontal, Connector_PinHeader_1.27mm:PinHeader_1x03_P1.27mm_Horizontal, F.Cu at (48.0, 95.0)
- added REF**: PinHeader_1x03_P1.00mm_Horizontal, Connector_PinHeader_1.00mm:PinHeader_1x03_P1.00mm_Horizontal, F.Cu at (41.2, 95.0)
- added REF**: DIP-4_W10.16mm_LongPads, Package_DIP:DIP-4_W10.16mm_LongPads, F.Cu at (23.0, 134.0)
- added REF**: DIP-4_W10.16mm, Package_DIP:DIP-4_W10.16mm, F.Cu at (23.0, 125.0)
- added REF**: DIP-4_W7.62mm_Socket, Package_DIP:DIP-4_W7.62mm_Socket, F.Cu at (24.0, 107.0)
- added REF**: DIP-4_W7.62mm_LongPads, Package_DIP:DIP-4_W7.62mm_LongPads, F.Cu at (24.0, 98.0)
- added REF**: DIP-4_W7.62mm_Socket_LongPads, Package_DIP:DIP-4_W7.62mm_Socket_LongPads, F.Cu at (24.0, 116.0)
- added REF**: DIP-4_W7.62mm, Package_DIP:DIP-4_W7.62mm, F.Cu at (24.0, 89.0)
- moved REF** 96.7 mm to (55.5, 28.0)
- moved REF** 96.7 mm to (48.0, 28.0)
- moved REF** 96.7 mm to (41.2, 28.0)
- moved REF** 96.7 mm to (23.0, 67.0)
- moved REF** 96.7 mm to (23.0, 58.0)
- moved REF** 96.7 mm to (24.0, 49.0)
- moved REF** 96.7 mm to (24.0, 40.0)
- moved REF** 96.7 mm to (24.0, 31.0)
- moved REF** 96.7 mm to (24.0, 22.0)
Routing:
- net (no net): track 120.0 -> 1440.0 mm
Other:
- board size 45 x 56 mm -> 258 x 176 mm

Commit message: adjust pcbNew
Parts:
- removed the REF** at (106.0, 158.5)
- removed the REF** at (28.0, 158.5)
- removed the REF** at (55.5, 28.0)
- removed the REF** at (48.0, 28.0)
- removed the REF** at (41.2, 28.0)
- removed the REF** at (23.0, 67.0)
- removed the REF** at (23.0, 58.0)
- removed the REF** at (24.0, 49.0)
- removed the REF** at (24.0, 40.0)
- removed the REF** at (24.0, 31.0)
- removed the REF** at (24.0, 22.0)
- removed the REF** at (28.0, 166.0)
- removed the REF** at (28.0, 172.8)
- removed the REF** at (67.0, 191.0)
- removed the REF** at (58.0, 191.0)
- removed the REF** at (40.0, 190.0)
- removed the REF** at (31.0, 190.0)
- removed the REF** at (49.0, 190.0)
- removed the REF** at (22.0, 190.0)
- removed the REF** at (268.5, 95.0)
- removed the REF** at (106.0, 166.0)
- removed the REF** at (261.0, 95.0)
- removed the REF** at (254.2, 95.0)
- removed the REF** at (236.0, 134.0)
- removed the REF** at (236.0, 125.0)
- removed the REF** at (237.0, 107.0)
- removed the REF** at (237.0, 98.0)
- removed the REF** at (237.0, 116.0)
- removed the REF** at (237.0, 89.0)
- removed the REF** at (268.5, 28.0)
- removed the REF** at (261.0, 28.0)
- removed the REF** at (106.0, 172.8)
- removed the REF** at (254.2, 28.0)
- removed the REF** at (236.0, 67.0)
- removed the REF** at (236.0, 58.0)
- removed the REF** at (237.0, 40.0)
- removed the REF** at (237.0, 31.0)
- removed the REF** at (237.0, 49.0)
- removed the REF** at (237.0, 22.0)
- removed the REF** at (215.5, 95.0)
- removed the REF** at (208.0, 95.0)
- removed the REF** at (201.2, 95.0)
- removed the REF** at (145.0, 191.0)
- removed the REF** at (183.0, 134.0)
- removed the REF** at (183.0, 125.0)
- removed the REF** at (184.0, 107.0)
- removed the REF** at (184.0, 98.0)
- removed the REF** at (184.0, 116.0)
- removed the REF** at (184.0, 89.0)
- removed the REF** at (215.5, 28.0)
- removed the REF** at (208.0, 28.0)
- removed the REF** at (201.2, 28.0)
- removed the REF** at (183.0, 67.0)
- removed the REF** at (136.0, 191.0)
- removed the REF** at (183.0, 58.0)
- removed the REF** at (184.0, 40.0)
- removed the REF** at (184.0, 31.0)
- removed the REF** at (184.0, 49.0)
- removed the REF** at (184.0, 22.0)
- removed the REF** at (118.0, 190.0)
- removed the REF** at (162.5, 28.0)
- removed the REF** at (155.0, 28.0)
- removed the REF** at (148.2, 28.0)
- removed the REF** at (130.0, 67.0)
- removed the REF** at (130.0, 58.0)
- removed the REF** at (131.0, 40.0)
- removed the REF** at (109.0, 190.0)
- removed the REF** at (131.0, 31.0)
- removed the REF** at (131.0, 49.0)
- removed the REF** at (131.0, 22.0)
- removed the REF** at (108.5, 95.0)
- removed the REF** at (101.0, 95.0)
- removed the REF** at (94.2, 95.0)
- removed the REF** at (76.0, 134.0)
- removed the REF** at (76.0, 125.0)
- removed the REF** at (77.0, 107.0)
- removed the REF** at (77.0, 98.0)
- removed the REF** at (127.0, 190.0)
- removed the REF** at (77.0, 116.0)
- removed the REF** at (77.0, 89.0)
- removed the REF** at (109.5, 28.0)
- removed the REF** at (102.0, 28.0)
- removed the REF** at (95.2, 28.0)
- removed the REF** at (77.0, 67.0)
- removed the REF** at (77.0, 58.0)
- removed the REF** at (78.0, 40.0)
- removed the REF** at (78.0, 31.0)
- removed the REF** at (78.0, 49.0)
- removed the REF** at (100.0, 190.0)
- removed the REF** at (78.0, 22.0)
- removed the REF** at (55.5, 95.0)
- removed the REF** at (48.0, 95.0)
- removed the REF** at (41.2, 95.0)
- removed the REF** at (23.0, 134.0)
- removed the REF** at (23.0, 125.0)
- removed the REF** at (24.0, 107.0)
- removed the REF** at (24.0, 98.0)
- removed the REF** at (24.0, 116.0)
- removed the REF** at (24.0, 89.0)
Routing:
- net (no net): track 1440.0 -> 120.0 mm
Other:
- board size 258 x 176 mm -> 45 x 56 mm
